File: hardware/layout/layout.kicad_pcb (KiCad board)
At the start: 4 copper layers, 50 x 20 mm, 72 parts, among them J1 HC-HDMI0019T-3, J2 GT-USB-7014G, Q1 2N7002, SW1 TS-1088-AR02016, U1 PCA9306DCUR, U2 AP2112K-3.3TRG1, U3 USBLC6-2SC6, U4 W25Q16JVSSIQ, U5 RP2040, Y1 X322512MSB4SI

Commit message: hardware: use board-level thermal overrides
Parts:
- TP20, TP21: footprint naorunaoru_picoarc_footprints_picoarc:TestPad_D1.0mm_Round_Thermal -> kicad_libraries_kicad-footprints_TestPoint@9.0.3:TestPoint_Pad_D1.0mm
- TP3, TP4: footprint naorunaoru_picoarc_footprints_picoarc:TestPad_1.0x1.0mm_RoundRect_Thermal -> naorunaoru_picoarc_footprints_picoarc:TestPad_1.0x1.0mm_RoundRect

Commit message: hardware: recover USB-powered DDC schematic and initial routing
Connections:
- R10 pad 2: HDMI._HDMI_5V -> VDD_5V
- R11 pad 2: HDMI._HDMI_5V -> VDD_5V
- R12 pad 1: HDMI._HDMI_5V -> VDD_5V
Routing:
- net HDMI._HDMI_5V: track 7.53 -> 6.23 mm, vias 3 -> 2
- net VDD_5V: track 10.4 -> 11.7 mm, vias 6 -> 7
Changed lines of the file:
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@@
 			(layers "F.Cu" "F.Mask" "F.Paste")
 			(roundrect_rratio 0.25)
-			(net "HDMI._HDMI_5V")
+			(net "VDD_5V")
 		)
 		(embedded_fonts no)
@@
 			(layers "F.Cu" "F.Mask" "F.Paste")
 			(roundrect_rratio 0.25)
-			(net "HDMI._HDMI_5V")
+			(net "VDD_5V")
 		)
 		(pad "2" smd roundrect
@@
 			(layers "F.Cu" "F.Mask" "F.Paste")
 			(roundrect_rratio 0.25)
-			(net "HDMI._HDMI_5V")
+			(net "VDD_5V")
 		)
 		(embedded_fonts no)
@@
 	)
 	(segment
-		(start 115.551401 110.96)
-		(end 116.1 110.96)
-		(width 0.16)
-		(layer "F.Cu")
-		(net "HDMI._HDMI_5V")
-	)
-	(segment
 		(start 117.25 106.72)
 		(end 118.2 106.72)
@@
 	)
 	(segment
-		(start 115.061401 111.45)
-		(end 115 111.45)
-		(width 0.16)
-		(layer "F.Cu")
-		(net "HDMI._HDMI_5V")
-	)
-	(segment
 		(start 116.77 107.21)
 		(end 116.3 107.68)
@@
 	)
 	(segment
-		(start 115.504248 111.007153)
-		(end 115.061401 111.45)
-		(width 0.16)
-		(layer "F.Cu")
-		(net "HDMI._HDMI_5V")
-	)
-	(segment
-		(start 115.504248 111.007153)
-		(end 115.551401 110.96)
-		(width 0.16)
-		(layer "F.Cu")
-		(net "HDMI._HDMI_5V")
-	)
-	(segment
 		(start 117.32 107.99)
 		(end 117.33 108)
@@
 	)
 	(via
-		(at 115.504248 111.007153)
-		(size 0.5)
-		(drill 0.3)
-		(layers "F.Cu" "B.Cu")
-		(net "HDMI._HDMI_5V")
-	)
-	(via
 		(at 112.392595 106.23037)
 		(size 0.5)
@@
 	)
 	(segment
+		(start 115.551401 110.96)
+		(end 116.1 110.96)
+		(width 0.16)
+		(layer "F.Cu")
+		(net "VDD_5V")
+	)
+	(segment
+		(start 115.061401 111.45)
+		(end 115 111.45)
+		(width 0.16)
+		(layer "F.Cu")
+		(net "VDD_5V")
+	)
+	(segment
 		(start 141.76 108.6)
 		(end 142.625 108.6)
@@
 	)
 	(segment
+		(start 115.504248 111.007153)
+		(end 115.061401 111.45)
+		(width 0.16)
+		(layer "F.Cu")
+		(net "VDD_5V")
+	)
+	(segment
+		(start 115.504248 111.007153)
+		(end 115.551401 110.96)
+		(width 0.16)
+		(layer "F.Cu")
+		(net "VDD_5V")
+	)
+	(segment
 		(start 137.230866 117.640932)
 		(end 137.893365 117.640932)
@@
 		(size 0.5)
 		(drill 0.3)
+		(layers "F.Cu" "B.Cu")
+		(net "VDD_5V")
+	)
+	(via
+		(at 115.504248 111.007153)
+		(size 0.5)
+		(drill 0.3)

Commit message: hardware: recover unfinished DDC layout from KiCad history
Parts:
- moved R7 7.08 mm to (114.0, 105.1), turned to 90 degrees
- moved R6 5.74 mm to (113.0, 106.2), turned to 90 degrees
- moved C2 5.34 mm to (116.1, 113.4), turned to 180 degrees
- moved R12 4.08 mm to (116.1, 112.4), turned to 0 degrees
- moved R13 3.66 mm to (117.3, 108.4), turned to 0 degrees
- moved R5 2.42 mm to (114.4, 107.0), turned to 0 degrees
- moved Q1 2.37 mm to (116.4, 105.8), turned to 180 degrees
- moved D3 0.66 mm to (111.6, 107.1), turned to -90 degrees
- moved R8 0.10 mm to (119.5, 108.5)
- moved C1 0.10 mm to (114.7, 114.5)
Routing:
- net HDMI_5V_SENSE: track 9.91 -> 17.0 mm
- net HDMI._HDMI_5V: track 6.23 -> 3.83 mm, vias 2 -> 0
- net HDMI._VREF2_EN: track 5.16 -> 3.19 mm
- net HPD_GATE: track 15.2 -> 13.4 mm
- net VDD_3V3: track 24.1 -> 22.2 mm, vias 17 -> 15
- net VDD_5V: track 11.7 -> 10.4 mm, vias 7 -> 6
- net GND: track 0.67 -> 0.00 mm, vias 47 -> 44
- removed copper zone on In2.Cu, net HDMI._HDMI_5V

Commit message: hardware: finish USB-powered DDC routing and document dual-role limits
Parts:
- moved R11 1.87 mm to (115.6, 108.7), turned to 0 degrees
- moved R13 0.30 mm to (117.6, 108.4)
- moved R8 0.10 mm to (119.4, 108.5)
Routing:
- net VDD_5V: track 10.4 -> 40.9 mm, vias 6 -> 8
- net VDD_3V3: track 22.2 -> 24.7 mm, vias 15 -> 16
- net DDC_SDA_5V: track 9.17 -> 10.3 mm
Changed lines of the file:
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@@
 	(footprint "kicad_libraries_kicad-footprints_Resistor_SMD@9.0.3:R_0402_1005Metric"
 		(layer "F.Cu")
-		(at 117.3 108.4)
+		(at 117.6 108.4)
 		(descr "Resistor SMD 0402 (1005 Metric), square (rectangular) end terminal, IPC-7351 nominal, (Body size source: IPC-SM-782 page 72, https://www.pcb-3d.com/wordpress/wp-content/uploads/ipc-sm-782a_amendment_1_and_2.pdf), generated with kicad-footprint-generator")
 		(tags "resistor")
@@
 	(footprint "kicad_libraries_kicad-footprints_Resistor_SMD@9.0.3:R_0402_1005Metric"
 		(layer "F.Cu")
-		(at 116.1 110.45 -90)
+		(at 115.6 108.65)
 		(descr "Resistor SMD 0402 (1005 Metric), square (rectangular) end terminal, IPC-7351 nominal, (Body size source: IPC-SM-782 page 72, https://www.pcb-3d.com/wordpress/wp-content/uploads/ipc-sm-782a_amendment_1_and_2.pdf), generated with kicad-footprint-generator")
 		(tags "resistor")
 		(property "Reference" "R11"
-			(at 0 1.315 90)
+			(at 0 1.315 180)
 			(layer "F.SilkS")
 			(hide yes)
@@
 		)
 		(property "Value" "0402WGF2201TCE"
-			(at 0 1.17 90)
+			(at 0 1.17 180)
 			(layer "F.Fab")
 			(hide yes)
@@
 		)
 		(property "Datasheet" ""
-			(at 0 0 90)
+			(at 0 0 180)
 			(layer "F.Fab")
 			(hide yes)
@@
 		)
 		(property "Description" "2.2k"
-			(at 0 0 90)
+			(at 0 0 180)
 			(layer "F.Fab")
 			(hide yes)
@@
 		)
 		(property "Path" "HDMI.R11.R"
-			(at 0 0 90)
+			(at 0 0 180)
 			(layer "F.SilkS")
 			(hide yes)
@@
 		)
 		(property "Manufacturer" "UNI-ROYAL(Uniroyal Elec)"
-			(at 0 0 90)
+			(at 0 0 180)
 			(layer "F.SilkS")
 			(hide yes)
@@
 		)
 		(property "Mpn" "0402WGF2201TCE"
-			(at 0 0 90)
+			(at 0 0 180)
 			(layer "F.SilkS")
 			(hide yes)
@@
 		)
 		(property "Package" "0402"
-			(at 0 0 90)
+			(at 0 0 180)
 			(layer "F.SilkS")
 			(hide yes)
@@
 		)
 		(property "Prefix" "R"
-			(at 0 0 90)
+			(at 0 0 180)
 			(layer "F.SilkS")
 			(hide yes)
@@
 		)
 		(property "Resistance" "2.2k"
-			(at 0 0 90)
+			(at 0 0 180)
 			(layer "F.SilkS")
 			(hide yes)
@@
 		)
 		(property "Type" "resistor"
-			(at 0 0 90)
+			(at 0 0 180)
 			(layer "F.SilkS")
 			(hide yes)
@@
 		(duplicate_pad_numbers_are_jumpers no)
 		(fp_line
-			(start -0.93 0.47)
-			(end -0.93 -0.47)
+			(start -0.93 -0.47)
+			(end 0.93 -0.47)
 			(stroke
 				(width 0.05)
@@
 		)
 		(fp_line
-			(start 0.93 0.47)
-			(end -0.93 0.47)
+			(start -0.93 0.47)
+			(end -0.93 -0.47)
 			(stroke
 				(width 0.05)
@@
 		)
 		(fp_line
-			(start -0.93 -0.47)
-			(end 0.93 -0.47)
+			(start 0.93 -0.47)
+			(end 0.93 0.47)
 			(stroke
 				(width 0.05)
@@
 		)
 		(fp_line
-			(start 0.93 -0.47)
-			(end 0.93 0.47)
+			(start 0.93 0.47)
+			(end -0.93 0.47)
 			(stroke
 				(width 0.05)
@@
 		)
 		(fp_line
-			(start -0.525 0.27)
-			(end -0.525 -0.27)
+			(start -0.525 -0.27)
+			(end 0.525 -0.27)
 			(stroke
 				(width 0.1)
@@
 		)
 		(fp_line
-			(start 0.525 0.27)
-			(end -0.525 0.27)
+			(start -0.525 0.27)
+			(end -0.525 -0.27)
 			(stroke
 				(width 0.1)
@@
 		)
 		(fp_line
-			(start -0.525 -0.27)
-			(end 0.525 -0.27)
+			(start 0.525 -0.27)
+			(end 0.525 0.27)
 			(stroke
 				(width 0.1)
@@
 		)
 		(fp_line
-			(start 0.525 -0.27)
-			(end 0.525 0.27)
+			(start 0.525 0.27)
+			(end -0.525 0.27)
 			(stroke
 				(width 0.1)
@@
 		)
 		(fp_text user "${REFERENCE}"
-			(at 0 0 90)
+			(at 0 0 180)
 			(layer "F.Fab")
 			(effects
@@
 		)
 		(pad "1" smd roundrect
-			(at -0.51 0 270)
+			(at -0.51 0)
 			(size 0.54 0.64)
 			(layers "F.Cu" "F.Mask" "F.Paste")
@@
 		)
 		(pad "2" smd roundrect
-			(at 0.51 0 270)
+			(at 0.51 0)
 			(size 0.54 0.64)
 			(layers "F.Cu" "F.Mask" "F.Paste")
@@
 	(footprint "kicad_libraries_kicad-footprints_Resistor_SMD@9.0.3:R_0402_1005Metric"
 		(layer "F.Cu")
-		(at 119.5 108.5 90)
+		(at 119.4 108.5 90)
 		(descr "Resistor SMD 0402 (1005 Metric), square (rectangular) end terminal, IPC-7351 nominal, (Body size source: IPC-SM-782 page 72, https://www.pcb-3d.com/wordpress/wp-content/uploads/ipc-sm-782a_amendment_1_and_2.pdf), generated with kicad-footprint-generator")
 		(tags "resistor")
@@
 	)
 	(segment
+		(start 118.11 108.4)
+		(end 118.52 107.99)
+		(width 0.25)
+		(layer "F.Cu")
+		(net "VDD_3V3")
+	)
+	(segment
 		(start 132.02 115.24)
 		(end 131.62 115.24)
@@
 	)
 	(segment
+		(start 118.52 107.99)
+		(end 120.4 107.99)
+		(width 0.25)
+		(layer "F.Cu")
+		(net "VDD_3V3")
+	)
+	(segment
 		(start 134.07 118.44)
 		(end 132.92 117.29)
@@
 	)
 	(via
+		(at 118.6 107.99)
+		(size 0.5)
+		(drill 0.3)
+		(layers "F.Cu" "B.Cu")
+		(net "VDD_3V3")
+	)
+	(via
 		(at 126.164888 116.945917)
 		(size 0.5)
@@
 	)
 	(segment
-		(start 116.79 107.31)
+		(start 117.09 107.01)
 		(end 117.3375 106.7625)
 		(width 0.16)
@@
 	)
 	(segment
-		(start 116.79 108.4)
-		(end 116.79 107.31)
+		(start 117.09 108.4)
+		(end 117.09 107.01)
 		(width 0.16)
 		(layer "F.Cu")
@@
 	)
 	(segment
-		(start 119.5 109.01)
+		(start 119.4 109.01)
 		(end 119.5 110.174999)
 		(width 0.16)
@@
 	)
 	(segment
+		(start 116.11 108.65)
+		(end 116.11 108.05)
+		(width 0.25)
+		(layer "F.Cu")
+		(net "VDD_5V")
+	)
+	(segment
 		(start 137.280865 115.740932)
 		(end 136.730865 115.190932)
@@
 	)
 	(segment
+		(start 115 111.45)
+		(end 115 112.4)
+		(width 0.25)
+		(layer "F.Cu")
+		(net "VDD_5V")
+	)
+	(segment
 		(start 141.76 108.6)
 		(end 142.625 108.6)
@@
 	)
 	(segment
+		(start 115 112.4)
+		(end 115.59 112.4)
+		(width 0.25)
+		(layer "F.Cu")
+		(net "VDD_5V")
+	)
+	(segment
 		(start 137.230866 117.640932)
 		(end 137.893365 117.640932)
@@
 	)
 	(via
+		(at 115 112.4)
+		(size 0.5)
+		(drill 0.3)
+		(layers "F.Cu" "B.Cu")
+		(net "VDD_5V")
+	)
+	(via
+		(at 116.11 108.05)
+		(size 0.5)
+		(drill 0.3)
+		(layers "F.Cu" "B.Cu")
+		(net "VDD_5V")
+	)
+	(via
 		(at 138.43 111.28)
 		(size 0.5)
@@
 	)
 	(segment
+		(start 115 112.4)
+		(end 115 111.2)
+		(width 0.3)
+		(layer "B.Cu")
+		(net "VDD_5V")
+	)
+	(segment
+		(start 115 111.2)
+		(end 117 109.2)
+		(width 0.3)
+		(layer "B.Cu")
+		(net "VDD_5V")
+	)
+	(segment
+		(start 116.11 108.05)
+		(end 116.11 110.09)
+		(width 0.3)
+		(layer "B.Cu")
+		(net "VDD_5V")
+	)
+	(segment
+		(start 135.9 109.2)
+		(end 137.38 110.68)
+		(width 0.3)
+		(layer "B.Cu")
+		(net "VDD_5V")
+	)
+	(segment
+		(start 117 109.2)
+		(end 135.9 109.2)
+		(width 0.3)
+		(layer "B.Cu")
+		(net "VDD_5V")
+	)
+	(segment
+		(start 137.38 110.68)
+		(end 137.83 110.68)
+		(width 0.3)
+		(layer "B.Cu")
+		(net "VDD_5V")
+	)
+	(segment
 		(start 139.96 116.97)
 		(end 140.12 117.13)
@@
 	)
 	(segment
+		(start 137.83 110.68)
+		(end 138.43 111.28)
+		(width 0.3)
+		(layer "B.Cu")
+		(net "VDD_5V")
+	)
+	(segment
 		(start 140.12 117.13)
 		(end 140.12 118.24)
@@
 	)
 	(segment
+		(start 115.09 109.81)
+		(end 115.09 108.65)
+		(width 0.16)
+		(layer "F.Cu")
+		(net "DDC_SDA_5V")
+	)
+	(segment
 		(start 114.472964 109.810001)
 		(end 115.970001 109.810001)
@@
 		)
 		(min_thickness 0.2)
-		(fill
+		(fill yes
 			(thermal_gap 0.25)
 			(thermal_bridge_width 0.3)
@@
 		)
 		(min_thickness 0.2)
-		(fill
+		(fill yes
 			(thermal_gap 0.25)
 			(thermal_bridge_width 0.3)
@@
 		)
 		(min_thickness 0.2)
-		(fill
+		(fill yes
 			(thermal_gap 0.25)
 			(thermal_bridge_width 0.3)
@@
 		)
 		(min_thickness 0.2)
-		(fill
+		(fill yes
 			(thermal_gap 0.25)
 			(thermal_bridge_width 0.3)
@@
 		)
 		(min_thickness 0.25)
-		(fill
+		(fill yes
 			(thermal_gap 0.5)
 			(thermal_bridge_width 0.5)
@@
 		)
 		(min_thickness 0.25)
-		(fill
+		(fill yes
 			(thermal_gap 0.5)
 			(thermal_bridge_width 0.5)
@@
 	)
 	(group "HDMI"
-		(members "030f12ec-625c-4962-82c8-f261731aabc0" "0883e297-18e7-4986-88f1-a3f0cf54a1fc"
-			"0e503c71-adf1-4932-be12-7efc19f42bfa" "0f363e8e-7d79-4c03-9199-90a3e2a79233"
-			"0f38ead5-3667-4a3a-9bca-327d03bf2f98" "15e0a97f-9044-4a91-ba39-869400f34a3d"
-			"1b954a77-2da6-4559-abfb-109195db3d36" "21ac0cac-7753-4714-a3b7-69fbb8ba667b"
-			"23da9bbd-ac06-46ef-9e5f-a8481e19c3a9" "27e25d70-c106-4c44-9345-e1f9f37718a8"
-			"400fffc6-ded0-4091-869f-90d82536f1cd" "51332b91-618b-4ef0-84a7-c8e239a11cc5"
-			"519452c5-6afd-46e7-8b11-3f0dd4337b9e" "5299f85e-6e27-46e4-ac77-20f59b7cc7d8"
-			"56253e14-0ba9-47d5-a2e6-f6ca39a309af" "58ea5bbd-5ecb-4841-8ad9-b6c745bb3453"
-			"5ba3a050-b094-4456-a275-f3e82d6c9859" "62e6dcf3-239f-4f98-ad82-2e230785ec33"
-			"6f72dcf1-4357-43aa-8b29-795dca3138a9" "7ba62d0f-c9d1-4f18-9e3f-1fdb75f63eb7"
+		(members "030f12ec-625c-4962-82c8-f261731aabc0" "03bb0866-0dc8-46e1-b52b-df12a2784162"
+			"0883e297-18e7-4986-88f1-a3f0cf54a1fc" "0e503c71-adf1-4932-be12-7efc19f42bfa"
+			"0f363e8e-7d79-4c03-9199-90a3e2a79233" "0f38ead5-3667-4a3a-9bca-327d03bf2f98"
+			"15e0a97f-9044-4a91-ba39-869400f34a3d" "1b954a77-2da6-4559-abfb-109195db3d36"
+			"21ac0cac-7753-4714-a3b7-69fbb8ba667b" "23da9bbd-ac06-46ef-9e5f-a8481e19c3a9"
+			"27e25d70-c106-4c44-9345-e1f9f37718a8" "400fffc6-ded0-4091-869f-90d82536f1cd"
+			"51332b91-618b-4ef0-84a7-c8e239a11cc5" "519452c5-6afd-46e7-8b11-3f0dd4337b9e"
+			"5299f85e-6e27-46e4-ac77-20f59b7cc7d8" "56253e14-0ba9-47d5-a2e6-f6ca39a309af"
+			"58ea5bbd-5ecb-4841-8ad9-b6c745bb3453" "5ba3a050-b094-4456-a275-f3e82d6c9859"
+			"62e6dcf3-239f-4f98-ad82-2e230785ec33" "6f72dcf1-4357-43aa-8b29-795dca3138a9"
+			"794fa290-f2a3-4e30-9572-7a0ac3ef9bfa" "7ba62d0f-c9d1-4f18-9e3f-1fdb75f63eb7"
 			"ad9edfbd-e358-4a49-b00f-bcc37390f923" "b2a7d150-31ba-41a4-90d0-74164664d68a"
 			"c1d478a8-d1a7-4725-ba5d-983c76674ee2" "c3d9abdf-0647-47b1-bc5b-9c536ea5066f"
